Commit message: Fix ROS2 mesh paths and RViz view

File: assets/environments/env_sldasm_export/urdf/env.urdf (robot description, URDF)
Before this commit: robot env_interaction, 3 links, 2 joints
Links:
- link base_link: geometry collision mesh filename=package://env_sldasm_export/meshes/base_link.STL; visual mesh filename=package://env_sldasm_export/meshes/base_link.STL
- link link1: geometry collision mesh filename=package://env_sldasm_export/meshes/link1.STL; visual mesh filename=package://env_sldasm_export/meshes/link1.STL
- link link2: geometry collision mesh filename=package://env_sldasm_export/meshes/link2.STL; visual mesh filename=package://env_sldasm_export/meshes/link2.STL

File: assets/environments/valve_parts/t_valve/urdf/model.urdf (robot description, URDF)
Before this commit: robot t_valve, 1 links, 0 joints
Links:
- link t_valve: geometry collision mesh filename=package://t_valve/meshes/T型阀.SLDPRT.STL; visual mesh filename=package://t_valve/meshes/T型阀.SLDPRT.STL

File: assets/environments/valve_parts/valve_1/urdf/model.urdf (robot description, URDF)
Before this commit: robot valve_1, 1 links, 0 joints
Links:
- link valve_1: geometry collision mesh filename=package://valve_1/meshes/1号阀.SLDPRT.STL; visual mesh filename=package://valve_1/meshes/1号阀.SLDPRT.STL

File: assets/environments/valve_parts/valve_2/urdf/model.urdf (robot description, URDF)
Before this commit: robot valve_2, 1 links, 0 joints
Links:
- link valve_2: geometry collision mesh filename=package://valve_2/meshes/2号阀件.SLDPRT.STL; visual mesh filename=package://valve_2/meshes/2号阀件.SLDPRT.STL
